File: fdmbox_pcb_tiny.kicad_pcb (KiCad board)
At the start: 2 copper layers, 128 parts, among them J1 POWER_IN, J10 T_ENV_IN, J11 POWER_OUT, J12 STP_SEL, J13 T_E0_OUT, J14 ICSP, J15 X0_MIN, J16 T_E1_OUT, J17 FAN_E0_OUT, J18 X1_MIN, J19 MOT_E1, J2 STP_SEL, J20 Y_MIN, J21 FAN_E1_OUT, J22 STP_SEL, J23 Z_MAX, J24 Z_MAX, J25 MOT_X0, J26 RPI_Conn, J27 BLTOUCH, J28 MOT_X1, J29 MOT_SPARE0, J3 T_E0_IN, J30 LOADCELL, J31 MOT_Y0, J32 STP_SEL, J33 RGB0, J34 MOT_Y1, J35 RGB1, J36 BED_PWM, J37 MOT_Z0, J38 MOT_SPARE1, J39 GP_PWM, J4 LFAN_E0_OUT, J40 MOT_Z1, J41 DBG_UART, J5 T_E1_IN, J6 LFAN_E1_OUT, J7 T_BED_IN, J8 FAN_ENV_OUT, J9 MOT_E0, Q1 BSS138, Q2 BSS138, Q3 STP55NF06L, Q4 STP55NF06L, Q5 STP55NF06L, Q6 STP55NF06L, Q7 STP55NF06L, Q8 BSS138, Q9 BSS138, SW1 RESET, U1 TSR_2-2450, U2 ATmega2560V-8AU, U3 PCA9531-Driver_LED, Y1 16MHz

Commit message: PCB finished -so far..
Parts:
- added REF**: MountingHole_3.2mm_M3_ISO14580_Pad, MountingHole:MountingHole_3.2mm_M3_ISO14580_Pad, F.Cu at (81.3, 142.2)
- added REF**: MountingHole_3.2mm_M3_ISO14580_Pad, MountingHole:MountingHole_3.2mm_M3_ISO14580_Pad, F.Cu at (81.3, 55.9)
- added REF**: MountingHole_3.2mm_M3_ISO14580_Pad, MountingHole:MountingHole_3.2mm_M3_ISO14580_Pad, F.Cu at (222.9, 55.9)
- added REF**: MountingHole_3.2mm_M3_ISO14580_Pad, MountingHole:MountingHole_3.2mm_M3_ISO14580_Pad, F.Cu at (223.5, 142.2)
- J23: value Z_MAX -> Z_MIN
- moved Q2 330.1 mm to (86.2, 99.2), turned to 270 degrees
- moved R5 320.0 mm to (87.8, 109.2), turned to 90 degrees
- moved Q1 318.1 mm to (89.9, 99.2), turned to 270 degrees
- moved F2 315.3 mm to (132.3, 120.9), turned to 90 degrees
- moved C3 309.8 mm to (102.5, 92.2), turned to 180 degrees
- moved C4 307.3 mm to (96.4, 102.2)
- moved R3 304.7 mm to (86.2, 95.1), turned to 180 degrees
- moved C6 301.2 mm to (100.3, 95.1), turned to 90 degrees
- moved C2 300.9 mm to (104.4, 121.0), turned to 270 degrees
- moved F1 295.2 mm to (136.1, 115.9), turned to 270 degrees
- moved F4 295.2 mm to (150.4, 121.9), turned to 270 degrees
- moved R28 295.0 mm to (126.9, 88.8), turned to 180 degrees
- moved R12 287.0 mm to (106.5, 88.8), turned to 180 degrees
- moved C7 280.0 mm to (119.6, 113.4)
- moved R4 279.8 mm to (87.8, 104.5), turned to 270 degrees
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Connections:
- J12 pad 1: +5V -> Net-(A2-Pad10)
- J12 pad 2: Net-(A2-Pad10) -> +5V
- J12 pad 3: +5V -> Net-(A2-Pad11)
- J12 pad 4: Net-(A2-Pad11) -> +5V
- J12 pad 5: +5V -> Net-(A2-Pad12)
- J12 pad 6: Net-(A2-Pad12) -> +5V
- J17 pad 2: GND -> +24V
- J2 pad 1: +5V -> Net-(A1-Pad10)
- J2 pad 2: Net-(A1-Pad10) -> +5V
- J2 pad 3: +5V -> Net-(A1-Pad11)
- J2 pad 4: Net-(A1-Pad11) -> +5V
- J2 pad 5: +5V -> Net-(A1-Pad12)
- J2 pad 6: Net-(A1-Pad12) -> +5V
- J21 pad 2: GND -> +24V
- J22 pad 1: +5V -> Net-(A3-Pad10)
- J22 pad 2: Net-(A3-Pad10) -> +5V
- J22 pad 3: +5V -> Net-(A3-Pad11)
- J22 pad 4: Net-(A3-Pad11) -> +5V
- J22 pad 5: +5V -> Net-(A3-Pad12)
- J22 pad 6: Net-(A3-Pad12) -> +5V
- J31 pad 1: /MOT_Y0_EN -> /MOT_Y_EN
- J31 pad 2: /MOT_Y0_DIR -> /MOT_Y_DIR
- J31 pad 3: /MOT_Y0_STEP -> /MOT_Y_STEP
- J32 pad 1: +5V -> Net-(A4-Pad10)
- J32 pad 2: Net-(A4-Pad10) -> +5V
- J32 pad 3: +5V -> Net-(A4-Pad11)
- J32 pad 4: Net-(A4-Pad11) -> +5V
- J32 pad 5: +5V -> Net-(A4-Pad12)
- J32 pad 6: Net-(A4-Pad12) -> +5V
- J34 pad 1: /MOT_Y1_EN -> /MOT_Y_EN
- J34 pad 2: /MOT_Y1_DIR -> /MOT_Y_DIR
- J34 pad 3: /MOT_Y1_STEP -> /MOT_Y_STEP
- J37 pad 1: /MOT_Z0_EN -> /MOT_Z_EN
- J37 pad 2: /MOT_Z0_DIR -> /MOT_Z_DIR
- J37 pad 3: /MOT_Z0_STEP -> /MOT_Z_STEP
- J40 pad 1: /MOT_Z1_EN -> /MOT_Z_EN
- J40 pad 2: /MOT_Z1_DIR -> /MOT_Z_DIR
- J40 pad 3: /MOT_Z1_STEP -> /MOT_Z_STEP
- R13 pad 1: GND -> +5V
- R21 pad 1: GND -> +5V
- R23 pad 1: GND -> +5V
- U2 pad 14: /GPPWM -> /BEDPWM
- U2 pad 15: /T_E0_L -> /F_E0_L
- U2 pad 16: /T_E1_L -> /F_E1_L
- U2 pad 17: /BEDPWM -> /T_E0_L
- U2 pad 18: /F_E0_L -> /T_E1_L
- U2 pad 19: /SPARE0_EN -> Net-(U2-Pad19)
- U2 pad 23: /BLTOUCH -> Net-(U2-Pad23)
- U2 pad 24: /SPARE1_STEP -> Net-(U2-Pad24)
- U2 pad 25: /SPARE1_DIR -> Net-(U2-Pad25)
- U2 pad 26: /SPARE1_EN -> Net-(U2-Pad26)
- U2 pad 27: /F_E1_L -> Net-(U2-Pad27)
- U2 pad 45: /X0MIN -> /LCELL
- U2 pad 46: /X1MIN -> /BLTOUCH
- U2 pad 47: /YMIN -> /X0MIN
- U2 pad 48: /ZMIN -> /ZMAX
- U2 pad 49: /ZMAX -> /ZMIN
- U2 pad 50: /LCELL -> /YMIN
- U2 pad 51: Net-(U2-Pad51) -> /X1MIN
- U2 pad 53: /MOT_Y0_STEP -> /MOT_Z_STEP
- U2 pad 54: /MOT_Y0_DIR -> /MOT_Z_DIR
- U2 pad 55: /MOT_Y0_EN -> /MOT_Z_EN
- U2 pad 56: /MOT_Y1_STEP -> /MOT_Y_STEP
- U2 pad 57: /MOT_Y1_DIR -> /MOT_Y_DIR
- U2 pad 58: /MOT_Y1_EN -> /MOT_Y_EN
- U2 pad 63: /MOT_Z0_EN -> /MOT_X0_STEP
- U2 pad 64: /MOT_Z0_DIR -> /MOT_X0_DIR
- U2 pad 65: /MOT_Z0_STEP -> /MOT_X0_EN
- U2 pad 66: /MOT_Z1_EN -> /MOT_X1_STEP
- U2 pad 67: /MOT_Z1_DIR -> /MOT_X1_DIR
- U2 pad 68: /MOT_Z1_STEP -> /MOT_X1_EN
- U2 pad 7: Net-(U2-Pad7) -> /GPPWM
- U2 pad 71: /SPARE0_DIR -> /SPARE1_DIR
- U2 pad 72: /SPARE0_STEP -> /SPARE1_STEP
- U2 pad 73: /E1_EN -> /SPARE1_EN
- U2 pad 74: /E1_DIR -> Net-(U2-Pad74)
- U2 pad 75: /E1_STEP -> Net-(U2-Pad75)
- U2 pad 76: /E0_EN -> /SPARE0_DIR
- U2 pad 77: /E0_DIR -> /SPARE0_STEP
- U2 pad 78: /E0_STEP -> /SPARE0_EN
- U2 pad 92: /MOT_X1_EN -> /E1_DIR
- U2 pad 93: /MOT_X1_DIR -> /E1_STEP
- U2 pad 94: /MOT_X1_STEP -> /E1_EN
- U2 pad 95: /MOT_X0_EN -> /E0_DIR
- U2 pad 96: /MOT_X0_DIR -> /E0_STEP
- U2 pad 97: /MOT_X0_STEP -> /E0_EN
Routing:
- net +24V: track 0.00 -> 524.5 mm, vias 0 -> 7
- net /T_E0_IN: track 0.00 -> 148.5 mm, vias 0 -> 2
- net /T_E1_IN: track 0.00 -> 141.4 mm, vias 0 -> 2
- net /ZMAX: track 0.00 -> 138.4 mm
- net /MOT_Z_STEP: track 0.00 -> 135.2 mm
- net /T_ENV_IN: track 0.00 -> 134.9 mm, vias 0 -> 2
- net /T_BED_IN: track 0.00 -> 133.6 mm, vias 0 -> 2
- net /MOT_Z_DIR: track 0.00 -> 132.5 mm
- net /MOT_Z_EN: track 0.00 -> 130.1 mm
- net /ZMIN: track 0.00 -> 128.8 mm
- net /LCELL: track 0.00 -> 128.2 mm
- net /MOT_Y_STEP: track 0.00 -> 120.6 mm
- net /BLTOUCH: track 0.00 -> 120.1 mm
- net /YMIN: track 0.00 -> 119.2 mm
- net /MOT_Y_DIR: track 0.00 -> 117.9 mm
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- added copper zone on 5V, net +5V
- added copper zone on B.Cu, net GND
- added copper zone on F.Cu, net GND
- added copper zone on In1.Cu, net GND
Other:
- board outline added: 152.4 x 96.5 mm
- copper layers 2 -> 4
